File: hardware/kicad/atmosmesh-room/atmosmesh-room.kicad_pcb (KiCad board)
At the start: 2 copper layers, 80 x 60 mm, 36 parts, among them U1 IDEASPARK_ESP32_1V14_TFT_30PIN

Commit message: :bug: fix(room): stop the schematic labelling the TFT pins as power rails
Final review of the generated artifacts. U1's nets were right, but its symbol
was still the bench project's ESP32_DevKit_V1_Socket, whose pin names run from
the opposite end of the row. KiCad writes each unconnected pad's own pin name
into a placeholder net, which is where this surfaced:

  pad 30  showed 3V3     - it is really GPIO23, the TFT MOSI line
  pad  4  showed GPIO34  - it is really GPIO12, the flash-voltage strap

That is precisely the hazard D-024 names: knowing the pin order makes the
socket more dangerous, because a builder can now confidently reach the wrong
pin. A schematic that prints "3V3" next to TFT MOSI is worse than a provisional
one that admits it does not know.

The symbol is renamed to Ideaspark_ESP32_1V14_TFT_30Pin and every pin relabelled
from IDEASPARK_PINS. Renaming needed three coordinated edits or KiCad refuses to
load the sheet at all: the entry name, each unit's own entry name, and the
library's default Value property.

The validator now refuses the DevKit name and asserts pads 30, 24, 4 and 10 are
labelled GPIO23/GPIO18/GPIO12/GPIO32 and left unconnected. Both mutation-proved:
relabelling pad 30 back to 3V3 fails, and connecting pad 24 fails.

Also completes the Zener inventory from the operator: 1N4733 through 1N4748.
The lowest is still 5.1 V and no 1N4728 is held, so the no-Zener rule now rests
on a complete list. Stale "60x80 mm" and "photos first" language cleared from
wiring.md and the silkscreen, since the build target is perfboard.

Gates: ERC 0, DRC 0 violations and 0 parity problems, both validators PASS,
git diff --check clean.
Other:
- board text added: "PARKED - PERFBOARD BUILD - DO NOT ORDER"
- board text removed: "DO NOT FABRICATE - PHOTOS FIRST"
Changed lines of the file:
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@@
 		(rev "PROVISIONAL A")
 		(company "AtmosMesh")
-		(comment 1 "DO NOT FABRICATE - exact module identities and pinouts unverified")
+		(comment 1 "PARKED - the build target is a 31x27 perfboard, not this board")
 	)
 	(layers
@@
 	(net 19 "SDS_TXD")
 	(net 20 "unconnected-(J_VEML-Pin_2-Pad2)")
-	(net 21 "unconnected-(U1-3V3-Pad30)")
-	(net 22 "unconnected-(U1-GND-Pad14)")
-	(net 23 "unconnected-(U1-GPIO1{slash}TX0-Pad18)")
-	(net 24 "unconnected-(U1-GPIO2-Pad27)")
-	(net 25 "unconnected-(U1-GPIO3{slash}RX0-Pad19)")
+	(net 21 "unconnected-(U1-EN-Pad15)")
+	(net 22 "unconnected-(U1-GPIO1-Pad28)")
+	(net 23 "unconnected-(U1-GPIO2-Pad19)")
+	(net 24 "unconnected-(U1-GPIO3-Pad27)")
+	(net 25 "unconnected-(U1-GPIO4-Pad20)")
 	(net 26 "unconnected-(U1-GPIO5-Pad23)")
-	(net 27 "unconnected-(U1-GPIO12-Pad12)")
-	(net 28 "unconnected-(U1-GPIO13-Pad13)")
-	(net 29 "unconnected-(U1-GPIO14-Pad11)")
-	(net 30 "unconnected-(U1-GPIO15-Pad28)")
-	(net 31 "unconnected-(U1-GPIO16{slash}RX2-Pad25)")
-	(net 32 "unconnected-(U1-GPIO17{slash}TX2-Pad24)")
-	(net 33 "unconnected-(U1-GPIO21-Pad20)")
-	(net 34 "unconnected-(U1-GPIO27-Pad10)")
-	(net 35 "unconnected-(U1-GPIO32-Pad6)")
-	(net 36 "unconnected-(U1-GPIO33-Pad7)")
-	(net 37 "unconnected-(U1-GPIO34-Pad4)")
-	(net 38 "unconnected-(U1-GPIO35-Pad5)")
-	(net 39 "unconnected-(U1-GPIO39{slash}VN-Pad3)")
-	(net 40 "unconnected-(U1-VIN-Pad15)")
+	(net 27 "unconnected-(U1-GPIO12-Pad4)")
+	(net 28 "unconnected-(U1-GPIO13-Pad3)")
+	(net 29 "unconnected-(U1-GPIO14-Pad5)")
+	(net 30 "unconnected-(U1-GPIO15-Pad18)")
+	(net 31 "unconnected-(U1-GPIO18-Pad24)")
+	(net 32 "unconnected-(U1-GPIO19-Pad25)")
+	(net 33 "unconnected-(U1-GPIO23-Pad30)")
+	(net 34 "unconnected-(U1-GPIO26-Pad7)")
+	(net 35 "unconnected-(U1-GPIO27-Pad6)")
+	(net 36 "unconnected-(U1-GPIO32-Pad10)")
+	(net 37 "unconnected-(U1-GPIO34-Pad12)")
+	(net 38 "unconnected-(U1-GPIO35-Pad11)")
+	(net 39 "unconnected-(U1-GPIO36-Pad14)")
+	(net 40 "unconnected-(U1-GPIO39-Pad13)")
 	(footprint "room:Ideaspark_30Pin_Provisional"
 		(layer "F.Cu")
@@
 			(layers "*.Cu" "*.Mask") (net 4 "GND") )
 		(pad "3" thru_hole circle (at 0.000 5.080) (size 1.7 1.7) (drill 0.8)
-			(layers "*.Cu" "*.Mask") (net 39 "unconnected-(U1-GPIO39{slash}VN-Pad3)") )
+			(layers "*.Cu" "*.Mask") (net 28 "unconnected-(U1-GPIO13-Pad3)") )
 		(pad "4" thru_hole circle (at 0.000 7.620) (size 1.7 1.7) (drill 0.8)
-			(layers "*.Cu" "*.Mask") (net 37 "unconnected-(U1-GPIO34-Pad4)") )
+			(layers "*.Cu" "*.Mask") (net 27 "unconnected-(U1-GPIO12-Pad4)") )
 		(pad "5" thru_hole circle (at 0.000 10.160) (size 1.7 1.7) (drill 0.8)
-			(layers "*.Cu" "*.Mask") (net 38 "unconnected-(U1-GPIO35-Pad5)") )
+			(layers "*.Cu" "*.Mask") (net 29 "unconnected-(U1-GPIO14-Pad5)") )
 		(pad "6" thru_hole circle (at 0.000 12.700) (size 1.7 1.7) (drill 0.8)
-			(layers "*.Cu" "*.Mask") (net 35 "unconnected-(U1-GPIO32-Pad6)") )
+			(layers "*.Cu" "*.Mask") (net 35 "unconnected-(U1-GPIO27-Pad6)") )
 		(pad "7" thru_hole circle (at 0.000 15.240) (size 1.7 1.7) (drill 0.8)
-			(layers "*.Cu" "*.Mask") (net 36 "unconnected-(U1-GPIO33-Pad7)") )
+			(layers "*.Cu" "*.Mask") (net 34 "unconnected-(U1-GPIO26-Pad7)") )
 		(pad "8" thru_hole circle (at 0.000 17.780) (size 1.7 1.7) (drill 0.8)
 			(layers "*.Cu" "*.Mask") (net 9 "GPIO25_BEEP") )
@@
 			(layers "*.Cu" "*.Mask") (net 10 "GPIO33_PIR_N") )
 		(pad "10" thru_hole circle (at 0.000 22.860) (size 1.7 1.7) (drill 0.8)
-			(layers "*.Cu" "*.Mask") (net 34 "unconnected-(U1-GPIO27-Pad10)") )
+			(layers "*.Cu" "*.Mask") (net 36 "unconnected-(U1-GPIO32-Pad10)") )
 		(pad "11" thru_hole circle (at 0.000 25.400) (size 1.7 1.7) (drill 0.8)
-			(layers "*.Cu" "*.Mask") (net 29 "unconnected-(U1-GPIO14-Pad11)") )
+			(layers "*.Cu" "*.Mask") (net 38 "unconnected-(U1-GPIO35-Pad11)") )
 		(pad "12" thru_hole circle (at 0.000 27.940) (size 1.7 1.7) (drill 0.8)
-			(layers "*.Cu" "*.Mask") (net 27 "unconnected-(U1-GPIO12-Pad12)") )
+			(layers "*.Cu" "*.Mask") (net 37 "unconnected-(U1-GPIO34-Pad12)") )
 		(pad "13" thru_hole circle (at 0.000 30.480) (size 1.7 1.7) (drill 0.8)
-			(layers "*.Cu" "*.Mask") (net 28 "unconnected-(U1-GPIO13-Pad13)") )
+			(layers "*.Cu" "*.Mask") (net 40 "unconnected-(U1-GPIO39-Pad13)") )
 		(pad "14" thru_hole circle (at 0.000 33.020) (size 1.7 1.7) (drill 0.8)
-			(layers "*.Cu" "*.Mask") (net 22 "unconnected-(U1-GND-Pad14)") )
+			(layers "*.Cu" "*.Mask") (net 39 "unconnected-(U1-GPIO36-Pad14)") )
 		(pad "15" thru_hole circle (at 0.000 35.560) (size 1.7 1.7) (drill 0.8)
-			(layers "*.Cu" "*.Mask") (net 40 "unconnected-(U1-VIN-Pad15)") )
+			(layers "*.Cu" "*.Mask") (net 21 "unconnected-(U1-EN-Pad15)") )
 		(pad "16" thru_hole circle (at 25.400 0.000) (size 1.7 1.7) (drill 0.8)
 			(layers "*.Cu" "*.Mask") (net 1 "+3V3") )
@@
 			(layers "*.Cu" "*.Mask") (net 4 "GND") )
 		(pad "18" thru_hole circle (at 25.400 5.080) (size 1.7 1.7) (drill 0.8)
-			(layers "*.Cu" "*.Mask") (net 23 "unconnected-(U1-GPIO1{slash}TX0-Pad18)") )
+			(layers "*.Cu" "*.Mask") (net 30 "unconnected-(U1-GPIO15-Pad18)") )
 		(pad "19" thru_hole circle (at 25.400 7.620) (size 1.7 1.7) (drill 0.8)
-			(layers "*.Cu" "*.Mask") (net 25 "unconnected-(U1-GPIO3{slash}RX0-Pad19)") )
+			(layers "*.Cu" "*.Mask") (net 23 "unconnected-(U1-GPIO2-Pad19)") )
 		(pad "20" thru_hole circle (at 25.400 10.160) (size 1.7 1.7) (drill 0.8)
-			(layers "*.Cu" "*.Mask") (net 33 "unconnected-(U1-GPIO21-Pad20)") )
+			(layers "*.Cu" "*.Mask") (net 25 "unconnected-(U1-GPIO4-Pad20)") )
 		(pad "21" thru_hole circle (at 25.400 12.700) (size 1.7 1.7) (drill 0.8)
 			(layers "*.Cu" "*.Mask") (net 5 "GPIO16_SDS_RX") )
@@
 			(layers "*.Cu" "*.Mask") (net 26 "unconnected-(U1-GPIO5-Pad23)") )
 		(pad "24" thru_hole circle (at 25.400 20.320) (size 1.7 1.7) (drill 0.8)
-			(layers "*.Cu" "*.Mask") (net 32 "unconnected-(U1-GPIO17{slash}TX2-Pad24)") )
+			(layers "*.Cu" "*.Mask") (net 31 "unconnected-(U1-GPIO18-Pad24)") )
 		(pad "25" thru_hole circle (at 25.400 22.860) (size 1.7 1.7) (drill 0.8)
-			(layers "*.Cu" "*.Mask") (net 31 "unconnected-(U1-GPIO16{slash}RX2-Pad25)") )
+			(layers "*.Cu" "*.Mask") (net 32 "unconnected-(U1-GPIO19-Pad25)") )
 		(pad "26" thru_hole circle (at 25.400 25.400) (size 1.7 1.7) (drill 0.8)
 			(layers "*.Cu" "*.Mask") (net 7 "GPIO21_SDA") )
 		(pad "27" thru_hole circle (at 25.400 27.940) (size 1.7 1.7) (drill 0.8)
-			(layers "*.Cu" "*.Mask") (net 24 "unconnected-(U1-GPIO2-Pad27)") )
+			(layers "*.Cu" "*.Mask") (net 24 "unconnected-(U1-GPIO3-Pad27)") )
 		(pad "28" thru_hole circle (at 25.400 30.480) (size 1.7 1.7) (drill 0.8)
-			(layers "*.Cu" "*.Mask") (net 30 "unconnected-(U1-GPIO15-Pad28)") )
+			(layers "*.Cu" "*.Mask") (net 22 "unconnected-(U1-GPIO1-Pad28)") )
 		(pad "29" thru_hole circle (at 25.400 33.020) (size 1.7 1.7) (drill 0.8)
 			(layers "*.Cu" "*.Mask") (net 8 "GPIO22_SCL") )
 		(pad "30" thru_hole circle (at 25.400 35.560) (size 1.7 1.7) (drill 0.8)
-			(layers "*.Cu" "*.Mask") (net 21 "unconnected-(U1-3V3-Pad30)") )
+			(layers "*.Cu" "*.Mask") (net 33 "unconnected-(U1-GPIO23-Pad30)") )
 	)
 	(footprint "room:PinHeader_1x05_P2.54mm"
@@
 	(gr_text "SHIELD FROM LCD" (at 113 66) (layer "F.SilkS")
 		(effects (font (size 0.8 0.8) (thickness 0.16)) (justify)) )
-	(gr_text "DO NOT FABRICATE - PHOTOS FIRST" (at 140 118.5) (layer "Dwgs.User")
+	(gr_text "PARKED - PERFBOARD BUILD - DO NOT ORDER" (at 140 118.5) (layer "Dwgs.User")
 		(effects (font (size 1.0 1.0) (thickness 0.16)) (justify)) )
 	(gr_rect (start 119 60.5) (end 155 67) (stroke (width 0.3) (type dash)) (fill none)

Commit message: :sparkles: feat(room): indicate live domains, and delete the switch the sensor makes unnecessary
Two improvements from the updated inventory, and one of them removes hardware
rather than adding it.

Domain indicators (D-029). Both 5 V jumpers are default-open and the build plan
requires them to stay open until measurements are recorded, but there was no way
to see whether a domain was live - on the one board in this project whose whole
risk story is an unverified 5 V rail. D_LED_3V3 (470R), D_LED_SDS and D_LED_PIR
(1k each) fix that. The 5 V indicators are fed downstream of their own jumpers,
so a lit LED is direct evidence that the jumper it reports on is closed. Red or
green only: a blue LED's ~3.0 V drop leaves 0.6 mA on the 3.3 V rail and reads
as dead.

ROOM-04 rewritten, and D-030 records why. It proposed an IRLZ34N low-side switch
to duty-cycle the SDS011 laser. That was wrong twice:

- The topology does not work. A low-side switch opens the ground return while
  VCC stays at 5 V, so the load is not de-powered - its ground floats up until
  current stops and the sensor sits partially biased. De-powering needs
  high-side switching and no P-channel part is in stock.
- It is unnecessary. nova-sds011.pdf lists "Manual hibernation" and "Timed
  hibernate (Cycle to work)" under Extended functionality, with sleep current
  under 4 mA annotated "Lase&Fan sleep". The sensor duty-cycles itself, and the
  operator's hard-wired TX leg already carries the command.

The parasitic path the old story worried about - TX2 idling HIGH into an
unpowered sensor - disappears with the switch. ROOM-04 is now a firmware story,
gated on obtaining Nova's separate control-protocol document rather than
guessing frame formats at a sensor.

Inventory also gains the HANTEK DSO2D15, IC sockets and heat shrink. The scope
matters: the SDS011 20 mV ripple check was written as "measure with an
oscilloscope" with no instrument on record, and the same tool can settle the
~200 pF bus-capacitance a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
Parts:
- added D_LED_3V3: LED RED 3V3 LIVE, room:D_Axial_P7.62mm, F.Cu at (123.0, 117.0)
- added D_LED_PIR: LED PIR 5V LIVE, room:D_Axial_P7.62mm, F.Cu at (162.0, 118.0)
- added D_LED_SDS: LED SDS 5V LIVE, room:D_Axial_P7.62mm, F.Cu at (154.0, 92.0)
- added R_LED_3V3: 470R, room:R_Axial_P7.62mm, F.Cu at (110.0, 117.0)
- added R_LED_PIR: 1k, room:R_Axial_P7.62mm, F.Cu at (152.0, 118.0)
- added R_LED_SDS: 1k, room:R_Axial_P7.62mm, F.Cu at (154.0, 88.0)
Other:
- board text added: "LED LIT = THAT 5V DOMAIN IS LIVE"

Commit message: :sparkles: feat(room): let the 5 V domain come from the bench supply instead of USB
The operator has a lab supply with adjustable voltage and current limit. That
changes the board, not just the procedure.

JP_5V_SRC is a 3-pin select feeding a new +5V_DOMAIN rail: shunt on 1-2 takes
the board's VIN, on 2-3 takes +5V_EXT from J_5V_EXT. JP_PIR_5V and JP_SDS_5V now
feed from +5V_DOMAIN rather than straight off VIN.

A 3-pin header accepts exactly one 2-pin shunt, so the two sources cannot be
bridged. Two independent 2-pin jumpers could both be closed and push the bench
supply back into the host's USB port. The generator refuses that arrangement and
refuses a domain wired straight to VIN; both mutation-proved.

This resolves an open blocker rather than measuring around it. spec-comparison.md
puts the USB rail near 650 mA peak coincidence before the SDS011 fan is added and
says 700 mA is not comfortable. With the external source selected the fan is not
on that rail at all.

Bring-up rule recorded in D-031: first power-up uses the external supply with the
current limit set just above the expected draw. A current-limited supply turns a
wiring error from a destroyed part into a supply that refuses to deliver - the
cheapest protection available to a project that has already lost an LDO once.

Also fixes a latent generator bug found on the way: silkscreen-vs-drawing layer
was chosen by a hard-coded index set, so every text inserted above position 8
silently moved a different label onto silkscreen. Layer is now stated per entry.

Gates: ERC 0, DRC 0 violations and 0 parity problems, both validators PASS,
git diff --check clean.
Parts:
- added JP_5V_SRC: SELECT: 1-2 USB / 2-3 EXT, room:PinHeader_1x03_P2.54mm, F.Cu at (119.0, 62.5)
- added J_5V_EXT: EXT 5V IN / GND, room:PinHeader_1x02_P2.54mm, F.Cu at (109.0, 62.5)
Connections:
- JP_PIR_5V pad 1: +5V_USB_CONFIRMED -> +5V_DOMAIN
- JP_SDS_5V pad 1: +5V_USB_CONFIRMED -> +5V_DOMAIN
- TP_5V pad 1: +5V_USB_CONFIRMED -> +5V_DOMAIN
Other:
- board text added: "5V SRC 1-2 USB 2-3 EXT"
